File: Hardware/SerialFusion/SerialFusion.kicad_sch (KiCad schematic)
At the start: 58 parts, among them J1 USB Type C, J2 ESP32_Prog, J3 UART_Debug, J4 120E_Sel, J5 RS232, J6 RS485, Q1 MMBT3904, Q2 MMBT3904, Q3 MMBT3904, SW1 EN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

Commit message: First stage design for Rev A is completed & files updated
Parts:
- added R21, R22: 4K7, Resistor_SMD:R_1206_3216Metric_Pad1.30x1.75mm_HandSolder, symbol Device:R_Small
- J5: footprint Connector_Dsub:DSUB-9_Pins_Horizontal_P2.77x2.84mm_EdgePinOffset9.40mm -> Connector_Dsub:DSUB-9_Socket_Horizontal_P2.77x2.84mm_EdgePinOffset14.56mm_Housed_MountingHolesOffset8.20mm
Connections:
- net +3.3V: now also R21.1, R22.1
- net +5VA: now also U3.3 (EN)
- net GND1: no longer U3.3 (EN)
- net Rx: now also R21.2
- net Tx: now also R22.2
Other:
- note added: "AUTO PROGRAMMER"
- note added: "ESP32 Prog."
- note added: "ISO Power Supply"
- note added: "RS232 CONVERTER"
- note added: "RS485 CONVERTER"
- note added: "UART DEBUG"
- note added: "USB(Type-C) to USART CONVERTER"
- moved on the sheet: C9
